File: Wifi_homesensor.kicad_sch (KiCad schematic)
At the start: 22 parts, among them J1 Pinhdr 3x2.5, U1 MCP16301, U2 WeMos_D1_mini, U3 SHT31-DIS

Commit message: schematic finished, pcb editing started
Parts:
- added C7: 100nF, Capacitor_SMD:C_0603_1608Metric, symbol Device:C_Small
- added D5: SM6T15A, Diode_SMD:D_SMB, symbol Diode:SM6T15A
- added F1: 100mA, Fuse:Fuse_1812_4532Metric, symbol Device:Polyfuse_Small
- added J2: Conn_01x02, TerminalBlock_Phoenix:TerminalBlock_Phoenix_MKDS-1,5-2-5.08_1x02_P5.08mm_Horizontal, symbol Connector_Generic:Conn_01x02
- added R8: 10k, Resistor_SMD:R_0603_1608Metric, symbol Device:R_Small
- added SW1: SW_Push, Button_Switch_THT:SW_Tactile_SPST_Angled_PTS645Vx83-2LFS, symbol Switch:SW_Push
- D3, D4: footprint (none) -> LED_SMD:LED_0805_2012Metric
Connections:
- net +12V: now also D5.1 (A1), F1.1
- net +3V3: now also C7.1, R8.2
- net GND: now also C7.2, D5.2 (A2), J2.1 (Pin_1), SW1.1
- net CONFIG: now reaches U2.3 (D0)
- net CONFIG: now also R8.1, SW1.2
- new net: F1.2, J2.2 (Pin_2)
Other:
- moved on the sheet: R4, R6

Commit message: pcb finished
Parts:
- added C8: 100uF 35V, Capacitor_THT:C_Radial_D8.0mm_H11.5mm_P3.50mm, symbol Device:C_Polarized_Small
- added FID1, FID2: Fiducial, Fiducial:Fiducial_0.75mm_Mask2.25mm, symbol Mechanical:Fiducial
- added LOGO1: Logo_Open_Hardware_Small, Symbol:OSHW-Logo2_14.6x12mm_SilkScreen, symbol Graphic:Logo_Open_Hardware_Small
- J2: value Conn_01x02 -> AK500/2
Connections:
- net +12V: now also C8.1
- net GND: now also J1.3 (Pin_3), C8.2; no longer J1.1 (Pin_1)
- net RX: now reaches U2.15 (RX)
- net RX: now also J1.2 (Pin_2); no longer J1.3 (Pin_3)
- net TX: now reaches U2.16 (TX)
- net TX: now also J1.1 (Pin_1); no longer J1.2 (Pin_2)
Other:
- note added: "Supply voltage 5...15V, limited by D5 MCP16301 works up to 30V"
- note added: "This is not used by ESPhome"
- moved on the sheet: D5, F1, J1, J2
